File: HARDWARE/Rele-Wifi.kicad_sch (KiCad schematic)
At the start: 42 parts, among them J3 Screw_Terminal_01x03, J4 Screw_Terminal_01x03, J5 Screw_Terminal_01x03, J6 Screw_Terminal_01x03, K3 Relay, K4 Relay, K5 Relay, K6 Relay, Q1 2N7002, Q2 2N7002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

Commit message: las quintillisas
pcb corregido
Parts:
- removed D1: LED, symbol Device:LED
- added C1: C_US, Capacitor_SMD:C_0805_2012Metric, symbol Device:C_US
- added C2: C, Capacitor_SMD:C_0805_2012Metric, symbol Device:C
- added J1: Screw_Terminal_01x02, TerminalBlock:TerminalBlock_MaiXu_MX126-5.0-02P_1x02_P5.00mm, symbol Connector:Screw_Terminal_01x02
- added U8: KA78M05_TO252, Package_TO_SOT_SMD:TO-252-2, symbol Regulator_Linear:KA78M05_TO252
- D10, D5, D6, D8: footprint Diode_SMD:D_0805_2012Metric -> Diode_SMD:D_SMA
Connections:
- net GND: now also Q1.2 (S), Q2.2 (S), Q3.2 (S), Q4.2 (S), R12.2, R16.2, R20.2, R24.2, J1.2 (Pin_2), U8.2 (GND)
- net GIO21: now reaches ESP32S1.6 (GPIO21)
- net GIO21: now also R9.2
- net +5V renamed 5V
- net 5V: now also C1.1
- net GIO23: no longer names the net of ESP32S1.2 (GPIO23)
- net GIO23: no longer R9.2
- new net: C2.1, J1.1 (Pin_1)
- new net: C2.2, U8.1 (VI)
- new net: C1.2, U8.3 (VO)

Commit message: 2,0
pcb terminado
Parts:
- added J2: Conn_01x04, Connector_PinSocket_2.54mm:PinSocket_1x05_P2.54mm_Vertical, symbol Connector_Generic:Conn_01x04
- added J7: Conn_01x08, Connector_PinSocket_2.54mm:PinSocket_1x08_P2.54mm_Vertical, symbol Connector_Generic:Conn_01x08
Connections:
- net 5V: now also U8.3 (VO)
- net GIO21: now also J2.3 (Pin_3); no longer R9.2
- net GIO22: now also J2.4 (Pin_4); no longer R13.2
- net GND: now also C1.2, C2.2, J2.1 (Pin_1), J7.8 (Pin_8)
- net 3,3V: now reaches ESP32S1.20 (3V3)
- net 3,3V: now also J2.2 (Pin_2), J7.7 (Pin_7)
- net GIO36: now reaches ESP32S1.22 (VP)
- net GIO36: now also J7.1 (Pin_1)
- net GIO39: now reaches ESP32S1.23 (VN)
- net GIO39: now also J7.2 (Pin_2)
- net GIO34: now reaches ESP32S1.24 (GPIO34)
- net GIO34: now also J7.3 (Pin_3)
- net GIO35: now reaches ESP32S1.25 (GPIO35)
- net GIO35: now also J7.4 (Pin_4)
- net GIO32: now reaches ESP32S1.26 (GPIO32)
- net GIO32: now also J7.5 (Pin_5)
- net GIO33: now reaches ESP32S1.27 (GPIO33)
- net GIO33: now also J7.6 (Pin_6)
- net GIO19: now reaches ESP32S1.8 (GPIO19)
- net GIO19: now also R13.2
- net GIO18: now reaches ESP32S1.9 (GPIO18)
- net GIO18: now also R9.2
- net at C2.1, J1.1 (Pin_1): now also U8.1 (VI)
Other:
- note added: "Alimentacion Y Regulacion"
- note added: "ESP32"
- note added: "Extenciones"
- note added: "Modulo 1"
- note added: "Modulo 2"
- note added: "Modulo 3"
- note added: "Modulo 4"
- title: (none) -> RELE-WIFI
- moved on the sheet: C1, C2, D3, D4, D7, D9, ESP32S1, J1, K3, K4, K5, K6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

Commit message: 3.0
END
Parts:
- U8: footprint Package_TO_SOT_SMD:TO-252-2 -> Package_TO_SOT_SMD:TO-263-3_TabPin2
Connections:
- net 3,3V: no longer J7.7 (Pin_7)
- net 5V: now also ESP32S1.38 (5V), J7.8 (Pin_8)
- net GND: now also J7.7 (Pin_7); no longer J7.8 (Pin_8)
Other:
- note added: "J.K.F"
Changed lines of the file:
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@@
 		)
 	)
+	(text "J.K.F"
+		(exclude_from_sim no)
+		(at 146.05 18.796 0)
+		(effects
+			(font
+				(face "Microsoft PhagsPa")
+				(size 5 5)
+				(thickness 0.254)
+				(bold yes)
+				(color 110 0 255 1)
+			)
+		)
+	)
 	(text "Alimentacion\nY\nRegulacion"
 		(exclude_from_sim no)
@@
 		)
 	)
-	(global_label "3,3V"
-		(shape input)
-		(at 160.02 147.32 270)
-		(fields_autoplaced yes)
-		(effects
-			(font
-				(size 1.27 1.27)
-				(thickness 0.254)
-				(bold yes)
-				(color 255 2 0 1)
-			)
-			(justify right)
-		)
-		(property "Intersheetrefs" "${INTERSHEET_REFS}"
-			(at 160.02 154.8936 90)
-			(effects
-				(font
-					(size 1.27 1.27)
-				)
-				(justify right)
-				(hide yes)
-			)
-		)
-	)
 	(global_label "GIO22"
 		(shape input)
@@
 	(global_label "3,3V"
 		(shape input)
-		(at 146.05 146.05 0)
+		(at 160.02 147.32 270)
 		(fields_autoplaced yes)
 		(effects
@@
 				(color 255 2 0 1)
 			)
-			(justify left)
+			(justify right)
 		)
 		(property "Intersheetrefs" "${INTERSHEET_REFS}"
-			(at 153.6236 146.05 0)
+			(at 160.02 154.8936 90)
 			(effects
 				(font
 					(size 1.27 1.27)
 				)
-				(justify left)
+				(justify right)
 				(hide yes)
 			)
@@
 		)
 	)
+	(global_label "5V"
+		(shape input)
+		(at 148.59 142.24 0)
+		(fields_autoplaced yes)
+		(effects
+			(font
+				(size 1.27 1.27)
+				(thickness 0.254)
+				(bold yes)
+			)
+			(justify left)
+		)
+		(property "Intersheetrefs" "${INTERSHEET_REFS}"
+			(at 154.3493 142.24 0)
+			(effects
+				(font
+					(size 1.27 1.27)
+				)
+				(justify left)
+				(hide yes)
+			)
+		)
+	)
 	(global_label "GIO19"
 		(shape input)
@@
 		)
 	)
+	(global_label "5V"
+		(shape input)
+		(at 135.89 100.33 180)
+		(fields_autoplaced yes)
+		(effects
+			(font
+				(size 1.27 1.27)
+				(thickness 0.254)
+				(bold yes)
+			)
+			(justify right)
+		)
+		(property "Intersheetrefs" "${INTERSHEET_REFS}"
+			(at 130.1307 100.33 0)
+			(effects
+				(font
+					(size 1.27 1.27)
+				)
+				(justify right)
+				(hide yes)
+			)
+		)
+	)
 	(global_label "COM-2"
 		(shape input)
@@
 	(symbol
 		(lib_id "power:GND")
-		(at 148.59 142.24 90)
+		(at 146.05 146.05 90)
 		(unit 1)
 		(exclude_from_sim no)
@@
 		(dnp no)
 		(property "Reference" "#PWR017"
-			(at 154.94 142.24 0)
+			(at 152.4 146.05 0)
 			(effects
 				(font
@@
 		)
 		(property "Value" "GND"
-			(at 151.892 141.478 0)
+			(at 149.352 145.288 0)
 			(effects
 				(font
@@
 		)
 		(property "Footprint" ""
-			(at 148.59 142.24 0)
+			(at 146.05 146.05 0)
 			(effects
 				(font
@@
 		)
 		(property "Datasheet" ""
-			(at 148.59 142.24 0)
+			(at 146.05 146.05 0)
 			(effects
 				(font
@@
 		)
 		(property "Description" "Power symbol creates a global label with name \"GND\" , ground"
-			(at 148.59 142.24 0)
+			(at 146.05 146.05 0)
 			(effects
 				(font
@@
 			)
 		)
-		(property "Footprint" "Package_TO_SOT_SMD:TO-252-2"
+		(property "Footprint" "Package_TO_SOT_SMD:TO-263-3_TabPin2"
 			(at 40.64 174.625 0)
 			(effects

Commit message: 4.0
Changed lines of the file:
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@@
 	)
 	(junction
-		(at 247.65 121.92)
-		(diameter 0)
-		(color 0 0 0 0)
-	)
-	(junction
 		(at 247.65 125.73)
 		(diameter 0)
@@
 	)
 	(junction
-		(at 73.66 49.53)
-		(diameter 0)
-		(color 0 0 0 0)
-	)
-	(junction
 		(at 237.49 36.83)
 		(diameter 0)
@@
 	(wire
 		(pts
-			(xy 130.81 71.12) (xy 129.54 71.12)
-		)
-		(stroke
-			(width 0)
-			(type default)
-		)
-	)
-	(wire
-		(pts
 			(xy 83.82 106.68) (xy 73.66 106.68)
 		)
@@
 	(wire
 		(pts
-			(xy 76.2 54.61) (xy 76.2 49.53)
+			(xy 76.2 54.61) (xy 76.2 53.34)
 		)
 		(stroke
@@
 	(wire
 		(pts
-			(xy 160.02 67.31) (xy 162.56 67.31)
+			(xy 160.02 67.31) (xy 163.83 67.31)
 		)
 		(stroke
@@
 	(wire
 		(pts
-			(xy 129.54 63.5) (xy 130.81 63.5)
-		)
-		(stroke
-			(width 0)
-			(type default)
-		)
-	)
-	(wire
-		(pts
 			(xy 269.24 146.05) (xy 261.62 146.05)
 		)
@@
 	(wire
 		(pts
-			(xy 250.19 127) (xy 250.19 121.92)
+			(xy 250.19 127) (xy 250.19 125.73)
 		)
 		(stroke
@@
 	(wire
 		(pts
-			(xy 133.35 59.69) (xy 129.54 59.69)
+			(xy 133.35 59.69) (xy 130.81 59.69)
 		)
 		(stroke
@@
 	(wire
 		(pts
-			(xy 73.66 41.91) (xy 73.66 49.53)
-		)
-		(stroke
-			(width 0)
-			(type default)
-		)
-	)
-	(wire
-		(pts
 			(xy 247.65 142.24) (xy 247.65 144.78)
 		)
@@
 	(wire
 		(pts
-			(xy 160.02 59.69) (xy 161.29 59.69)
+			(xy 160.02 59.69) (xy 163.83 59.69)
 		)
 		(stroke
@@
 	(wire
 		(pts
-			(xy 162.56 71.12) (xy 165.1 71.12)
+			(xy 162.56 71.12) (xy 163.83 71.12)
 		)
 		(stroke
@@
 	(wire
 		(pts
-			(xy 162.56 83.82) (xy 165.1 83.82)
+			(xy 162.56 83.82) (xy 163.83 83.82)
 		)
 		(stroke
@@
 	(wire
 		(pts
-			(xy 247.65 121.92) (xy 247.65 125.73)
-		)
-		(stroke
-			(width 0)
-			(type default)
-		)
-	)
-	(wire
-		(pts
 			(xy 162.56 72.39) (xy 162.56 71.12)
 		)
@@
 	(wire
 		(pts
-			(xy 250.19 121.92) (xy 247.65 121.92)
+			(xy 250.19 125.73) (xy 247.65 125.73)
 		)
 		(stroke
@@
 	(wire
 		(pts
-			(xy 247.65 114.3) (xy 247.65 121.92)
+			(xy 247.65 114.3) (xy 247.65 125.73)
 		)
 		(stroke
@@
 	(wire
 		(pts
-			(xy 73.66 49.53) (xy 73.66 53.34)
+			(xy 73.66 41.91) (xy 73.66 53.34)
 		)
 		(stroke
@@
 	(wire
 		(pts
-			(xy 133.35 52.07) (xy 132.08 52.07)
+			(xy 133.35 52.07) (xy 129.54 52.07)
 		)
 		(stroke
@@
 	(wire
 		(pts
-			(xy 160.02 74.93) (xy 161.29 74.93)
+			(xy 160.02 74.93) (xy 163.83 74.93)
 		)
 		(stroke
@@
 	(wire
 		(pts
-			(xy 76.2 49.53) (xy 73.66 49.53)
+			(xy 76.2 53.34) (xy 73.66 53.34)
 		)
 		(stroke
@@
 	(wire
 		(pts
-			(xy 129.54 67.31) (xy 135.89 67.31)
+			(xy 130.81 67.31) (xy 135.89 67.31)
 		)
 		(stroke
@@
 	(global_label "GIO21"
 		(shape input)
-		(at 162.56 67.31 0)
+		(at 163.83 67.31 0)
 		(fields_autoplaced yes)
 		(effects
@@
 		)
 		(property "Intersheetrefs" "${INTERSHEET_REFS}"
-			(at 171.6455 67.31 0)
+			(at 172.9155 67.31 0)
 			(effects
 				(font
@@
 	(global_label "GIO35"
 		(shape input)
-		(at 129.54 67.31 180)
+		(at 130.81 67.31 180)
 		(fields_autoplaced yes)
 		(effects
@@
 		)
 		(property "Intersheetrefs" "${INTERSHEET_REFS}"
-			(at 120.4545 67.31 0)
+			(at 121.7245 67.31 0)
 			(effects
 				(font
@@
 	(global_label "GIO18"
 		(shape input)
-		(at 161.29 74.93 0)
+		(at 163.83 74.93 0)
 		(fields_autoplaced yes)
 		(effects
@@
 		)
 		(property "Intersheetrefs" "${INTERSHEET_REFS}"
-			(at 170.3755 74.93 0)
+			(at 172.9155 74.93 0)
 			(effects
 				(font
@@
 	(global_label "GIO16"
 		(shape input)
-		(at 165.1 83.82 0)
+		(at 163.83 83.82 0)
 		(fields_autoplaced yes)
 		(effects
@@
 		)
 		(property "Intersheetrefs" "${INTERSHEET_REFS}"
-			(at 174.1855 83.82 0)
+			(at 172.9155 83.82 0)
 			(effects
 				(font
@@
 	(global_label "GIO22"
 		(shape input)
-		(at 161.29 59.69 0)
+		(at 163.83 59.69 0)
 		(fields_autoplaced yes)
 		(effects
@@
 		)
 		(property "Intersheetrefs" "${INTERSHEET_REFS}"
-			(at 170.3755 59.69 0)
+			(at 172.9155 59.69 0)
 			(effects
 				(font
@@
 	(global_label "GIO19"
 		(shape input)
-		(at 165.1 71.12 0)
+		(at 163.83 71.12 0)
 		(fields_autoplaced yes)
 		(effects
@@
 		)
 		(property "Intersheetrefs" "${INTERSHEET_REFS}"
-			(at 174.1855 71.12 0)
+			(at 172.9155 71.12 0)
 			(effects
 				(font
@@
 	(global_label "3,3V"
 		(shape input)
-		(at 132.08 52.07 180)
+		(at 129.54 52.07 180)
 		(fields_autoplaced yes)
 		(effects
@@
 		)
 		(property "Intersheetrefs" "${INTERSHEET_REFS}"
-			(at 124.5064 52.07 0)
+			(at 121.9664 52.07 0)
 			(effects
 				(font
@@
 	(global_label "GIO32"
 		(shape input)
-		(at 129.54 71.12 180)
+		(at 130.81 71.12 180)
 		(fields_autoplaced yes)
 		(effects
@@
 		)
 		(property "Intersheetrefs" "${INTERSHEET_REFS}"
-			(at 120.4545 71.12 0)
+			(at 121.7245 71.12 0)
 			(effects
 				(font
@@
 	(global_label "GIO34"
 		(shape input)
-		(at 129.54 63.5 180)
+		(at 130.81 63.5 180)
 		(fields_autoplaced yes)
 		(effects
@@
 		)
 		(property "Intersheetrefs" "${INTERSHEET_REFS}"
-			(at 120.4545 63.5 0)
+			(at 121.7245 63.5 0)
 			(effects
 				(font
@@
 	(global_label "GIO39"
 		(shape input)
-		(at 129.54 59.69 180)
+		(at 130.81 59.69 180)
 		(fields_autoplaced yes)
 		(effects
@@
 		)
 		(property "Intersheetrefs" "${INTERSHEET_REFS}"
-			(at 120.4545 59.69 0)
+			(at 121.7245 59.69 0)
 			(effects
 				(font

Commit message: CAMBIO DE HUELLA
Parts:
- U8: footprint Package_TO_SOT_SMD:TO-263-3_TabPin2 -> Package_TO_SOT_SMD:TO-263-2
Changed lines of the file:
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@@
 			)
 		)
-		(property "Footprint" "Package_TO_SOT_SMD:TO-263-3_TabPin2"
+		(property "Footprint" "Package_TO_SOT_SMD:TO-263-2"
 			(at 40.64 174.625 0)
 			(effects
